File: surface-mount/kicad/badge.kicad_pcb (KiCad board)
At the start: 2 copper layers, 76.2 x 113 mm, 99 parts, among them U1 ATtiny85-20SF, U2 CD4021B, U3 SN74HC595, U4 SN74HC595

Commit message: Update badge
Signed-off-by: Josh Bressers <josh@bress.net>
Parts:
- added G***: LOGO, LOGO, F.Cu at (198.8, 93.6)
- added G***: LOGO, LOGO, B.Cu at (190.6, 91.7)
- moved R10 17.9 mm to (215.5, 80.8)
- moved R13 17.9 mm to (215.5, 70.6)
- moved R15 17.9 mm to (215.5, 75.7)
- moved R16 17.9 mm to (215.5, 73.2)
- moved R9 17.9 mm to (215.5, 78.2)
- moved R11 17.9 mm to (215.5, 83.3)
- moved R12 17.9 mm to (215.5, 85.9)
- moved R14 17.9 mm to (215.5, 68.1)
Routing:
- net Net-(U2-D2): track 118.9 -> 138.4 mm
- net Net-(U2-D4): track 125.3 -> 144.7 mm
- net Net-(U2-D6): track 92.6 -> 111.9 mm
- net Net-(U2-D7): track 90.9 -> 110.2 mm
- net Net-(U2-D0): track 116.5 -> 135.9 mm
- net Net-(U2-D1): track 108.4 -> 127.8 mm
- net Net-(U2-D5): track 121.5 -> 140.9 mm
- net Net-(U2-D3): track 108.4 -> 127.8 mm
- net GND: track 202.6 -> 204.3 mm
Other:
- board text added: "This badge is hackable github.com/OpenBadgeProject"
- board text added: "grassr00tz.com"
- board text removed: "This badge is hackable github.com/joshbressers/badge"
